Commit message: bro lafda fixed

File: assets/camera.urdf (robot description, URDF)
Before this commit: robot simple_robot, 4 links, 3 joints
Links:
- removed link cam_left
- removed link cam_right
- added link cam_neg; visual box size=0.05 0.05 0.05
- added link cam_pos; visual box size=0.05 0.05 0.05
Joints:
- removed joint cam_left_yaw
- removed joint cam_right_yaw
- added joint cam_neg_yaw: type revolute, parent h_rod, child cam_neg, origin xyz=-0.08125 0 0.04 rpy=0 0 0, axis 0 0 1, limit lower=-3.14 upper=3.14 effort=10 velocity=1
- added joint cam_pos_yaw: type revolute, parent h_rod, child cam_pos, origin xyz=0.08125 0 0.04 rpy=0 0 0, axis 0 0 1, limit lower=-3.14 upper=3.14 effort=10 velocity=1

File: assets/camera.xacro (robot description, xacro)
@@ -12,5 +12,5 @@
   <link name="base_link"/>
   <link name="h_rod"/>
-  <link name="cam_left">
+  <link name="cam_neg">
     <visual>
       <geometry>
@@ -22,5 +22,5 @@
     </visual>
   </link>
-  <link name="cam_right">
+  <link name="cam_pos">
     <visual>
       <geometry>
@@ -40,14 +40,14 @@
     <limit lower="${joint_limit_lower}" upper="${joint_limit_upper}" effort="${joint_effort}" velocity="${joint_velocity}"/>
   </joint>
-  <joint name="cam_left_yaw" type="revolute">
+  <joint name="cam_neg_yaw" type="revolute">
     <parent link="h_rod"/>
-    <child link="cam_left"/>
+    <child link="cam_neg"/>
     <origin xyz="-${baseline/2} 0 ${camera_stalk_height}" rpy="0 0 0"/>
     <axis xyz="0 0 1"/>
     <limit lower="${joint_limit_lower}" upper="${joint_limit_upper}" effort="${joint_effort}" velocity="${joint_velocity}"/>
   </joint>
-  <joint name="cam_right_yaw" type="revolute">
+  <joint name="cam_pos_yaw" type="revolute">
     <parent link="h_rod"/>
-    <child link="cam_right"/>
+    <child link="cam_pos"/>
     <origin xyz="${baseline/2} 0 ${camera_stalk_height}" rpy="0 0 0"/>
     <axis xyz="0 0 1"/>

Commit message: backup2

File: assets/camera.urdf (robot description, URDF)
Before this commit: robot simple_robot, 4 links, 3 joints
Joints:
- joint cam_neg_yaw: origin xyz=-0.08125 0 0.04 rpy=0 0 0 -> xyz=0.08125 0 0.04 rpy=0 0 0
- joint cam_pos_yaw: origin xyz=0.08125 0 0.04 rpy=0 0 0 -> xyz=-0.08125 0 0.04 rpy=0 0 0
